Commit message: add livox mid360 lidar

File: skid4wd_description/urdf/skid4wd.xacro (robot description, xacro)
@@ -73,4 +73,64 @@
   </sensor>
 </gazebo>
+<!-- Livox MID-360 LiDAR link definition -->
+<link name="lidar_link">
+  <inertial>
+    <origin rpy="0 0 0" xyz="0 0 0"/>
+    <mass value="0.5"/> <!-- 假设的质量，可以根据实际情况调整 -->
+    <inertia ixx="0.002" ixy="0.0" ixz="0.0" iyy="0.002" iyz="0.0" izz="0.002"/>
+  </inertial>
+  <visual>
+    <origin xyz="0 0 -0.03" rpy="1.57 0 3.14"/>
+    <geometry>
+      <mesh filename="package://skid4wd_description/meshes/livox-mid360.dae">
+      </mesh>
+    </geometry>
+  </visual>
+  <collision>
+    <origin rpy="0 0 -0.03" xyz="0 0 3.14"/>
+    <geometry>
+      <box size="0.1 0.1 0.15"/>
+    </geometry>
+  </collision>
+</link>
+<!-- LiDAR Joint definition -->
+<joint name="lidar_joint" type="fixed">
+  <parent link="base_link"/>
+  <child link="lidar_link"/>
+  <origin xyz="0 0 0.2" rpy="0 0 0"/> <!-- 设置LiDAR的位置，您可以根据需要调整高度 -->
+</joint>
+<!-- LiDAR plugin configuration -->
+<gazebo reference="lidar_link">
+  <sensor type="ray" name="lidar_sensor">
+    <pose>0 0 0 0 0 0</pose>
+    <visualize>false</visualize>
+    <update_rate>10</update_rate>
+    <ray>
+      <scan>
+        <horizontal>
+          <samples>360</samples>
+          <resolution>1</resolution>
+          <min_angle>-1.57</min_angle>
+          <max_angle>1.57</max_angle>
+        </horizontal>
+        <vertical>
+          <samples>30</samples>
+          <resolution>1</resolution>
+          <min_angle>-0.3</min_angle>
+          <max_angle>0.3</max_angle>
+        </vertical>
+      </scan>
+      <range>
+        <min>0.1</min>
+        <max>100</max>
+        <resolution>0.01</resolution>
+      </range>
+    </ray>
+    <plugin name="gazebo_ros_lidar" filename="libgazebo_ros_laser.so">
+      <topicName>/livox/lidar/scan</topicName> <!-- 发布的激光雷达话题 -->
+      <frameName>lidar_link</frameName>
+    </plugin>
+  </sensor>
+</gazebo>
 <link name="wheel_front_left_1">
   <inertial>

Commit message: add D435

File: skid4wd_description/urdf/skid4wd.xacro (robot description, xacro)
@@ -4,4 +4,6 @@
 <xacro:include filename="$(find skid4wd_description)/urdf/skid4wd.trans" />
 <xacro:include filename="$(find skid4wd_description)/urdf/skid4wd.gazebo" />
+<xacro:include filename="$(find realsense_ros_gazebo)/xacro/tracker.xacro"/>
+<xacro:include filename="$(find realsense_ros_gazebo)/xacro/depthcam.xacro"/>
 <xacro:property name="PI" value="3.14"/>
 <!-- Base link definition -->
@@ -29,5 +31,5 @@
 <link name="imu_link">
   <inertial>
-    <origin rpy="0 0 0" xyz="0 0 0"/>
+    <origin rpy="0 0 0.02" xyz="0 0 0"/>
     <mass value="0.1"/>
     <inertia ixx="0.001" ixy="0.0" ixz="0.0" iyy="0.001" iyz="0.0" izz="0.001"/>
@@ -36,5 +38,5 @@
     <origin rpy="0 0 0" xyz="0 0 0"/>
     <geometry>
-      <cylinder length="0.1" radius="0.02"/>
+      <cylinder length="0.01" radius="0.02"/>
     </geometry>
     <material name="blue"/>
@@ -43,5 +45,5 @@
     <origin rpy="0 0 0" xyz="0 0 0"/>
     <geometry>
-      <cylinder length="0.1" radius="0.02"/>
+      <cylinder length="0.01" radius="0.02"/>
     </geometry>
   </collision>
@@ -51,5 +53,5 @@
   <parent link="base_link"/>
   <child link="imu_link"/>
-  <origin xyz="0.1 0 0.1" rpy="0 0 0"/>
+  <origin xyz="0 0 0" rpy="0 0 0"/>
 </joint>
 <!-- IMU plugin for 'body_link' -->
@@ -73,5 +75,8 @@
   </sensor>
 </gazebo>
-<!-- Livox MID-360 LiDAR link definition -->
+<xacro:realsense_d435 sensor_name="d435" parent_link="base_link" rate="10">
+<origin rpy="0 0 0 " xyz="0.27 0 0.09"/>
+</xacro:realsense_d435>
+<!-- LiDAR link definition -->
 <link name="lidar_link">
   <inertial>

Commit message: add uneven model

File: skid4wd_description/urdf/skid4wd.xacro (robot description, xacro)
@@ -40,5 +40,7 @@
       <cylinder length="0.01" radius="0.02"/>
     </geometry>
-    <material name="blue"/>
+    <material name="white">
+      <color rgba="1 1 1 1"/>  <!-- 直接定义颜色 -->
+    </material>
   </visual>
   <collision>
@@ -217,4 +219,12 @@
     </geometry>
   </collision>
+  <!-- Rear Right Wheel Force Sensor -->
+  <plugin name="force_sensor_plugin" filename="libgazebo_ros_force_torque_sensor.so">
+    <robotNamespace>/robot</robotNamespace>
+    <sensor_name>force_sensor_rear_right</sensor_name>   <!-- 传感器名称 -->
+    <topic_name>/skid4wd/rear_right_force</topic_name>   <!-- 发布力数据的ROS话题 -->
+    <frame>wheel_rear_right_1</frame>                     <!-- 传感器参考框架 -->
+    <update_rate>1000</update_rate>                       <!-- 传感器的更新频率 -->
+  </plugin>
 </link>
 <joint name="joint_front_left" type="continuous">

Commit message: git contact data

File: skid4wd_description/urdf/skid4wd.xacro (robot description, xacro)
@@ -144,5 +144,5 @@
     <origin rpy="0 0 0" xyz="2.3943220794908626e-08 -0.009939147977344326 -1.8492763799449197e-08"/>
     <mass value="0.552895033700559"/>
-    <inertia ixx="0.001246" ixy="0.0" ixz="-0.0" iyy="0.002096" iyz="-0.0" izz="0.001246"/>
+    <inertia ixx="0.001246" ixy="0.0" ixz="0.0" iyy="0.002096" iyz="0.0" izz="0.001246"/>
   </inertial>
   <visual>
@@ -219,12 +219,4 @@
     </geometry>
   </collision>
-  <!-- Rear Right Wheel Force Sensor -->
-  <plugin name="force_sensor_plugin" filename="libgazebo_ros_force_torque_sensor.so">
-    <robotNamespace>/robot</robotNamespace>
-    <sensor_name>force_sensor_rear_right</sensor_name>   <!-- 传感器名称 -->
-    <topic_name>/skid4wd/rear_right_force</topic_name>   <!-- 发布力数据的ROS话题 -->
-    <frame>wheel_rear_right_1</frame>                     <!-- 传感器参考框架 -->
-    <update_rate>1000</update_rate>                       <!-- 传感器的更新频率 -->
-  </plugin>
 </link>
 <joint name="joint_front_left" type="continuous">
