Commit message: add force mark

File: willand_description/urdf/carmodel2.urdf (robot description, URDF)
Before this commit: robot carmodel, 7 links, 6 joints
Links:
- removed link base_footprint
- removed link base_scan
- link base_link: geometry collision box size=0.5 0.3 0.07; visual mesh filename=package://willand_description/meshes/Body.STL
Joints:
- removed joint base_footprint_joint
- removed joint scan_joint

File: willand_description/urdf/carmodel2.urdf.xacro (robot description, xacro)
@@ -1,4 +1,4 @@
 <?xml version="1.0"?>
-<robot name="carmodel" xmlns:xacro="http://ros.org/wiki/xacro">
+<robot name="willand" xmlns:xacro="http://ros.org/wiki/xacro">
   <xacro:include filename="$(find willand_description)/urdf/carmodel2.urdf"/>
   <xacro:property name="wheel_radius" value="0.03018"/>
@@ -59,59 +59,4 @@
     </plugin>
   </gazebo>
-  <gazebo>
-    <plugin name="differential_drive_controller" filename="libgazebo_ros_diff_drive.so">
-      <rosDebugLevel>na</rosDebugLevel>
-      <publishWheelTF>true</publishWheelTF>
-      <robotNamespace>/</robotNamespace>
-      <publishTf>true</publishTf>
-      <publishWheelJointState>true</publishWheelJointState>
-      <alwaysOn>true</alwaysOn>
-      <updateRate>30.0</updateRate>
-      <legacyMode>true</legacyMode>
-      <leftJoint>joint_base_wheel1</leftJoint>
-      <rightJoint>joint_base_wheel3</rightJoint>
-      <wheelSeparation>${width*2}</wheelSeparation>
-      <wheelDiameter>${2*wheel_radius}</wheelDiameter>
-      <broadcastTF>1</broadcastTF>
-      <wheelTorque>50</wheelTorque>
-      <wheelAcceleration>1.8</wheelAcceleration>
-      <commandTopic>cmd_vel</commandTopic>
-      <odometryFrame>odom</odometryFrame>
-      <odometryTopic>odom</odometryTopic>
-      <odometrySource>world</odometrySource>
-      <robotBaseFrame>base_footprint</robotBaseFrame>
-    </plugin>
-  </gazebo>
-  <gazebo reference="base_scan">
-    <sensor type="ray" name="lds_lfcd_sensor">
-    <pose>0 0 0.1 0 0 0</pose>
-    <visualize>false</visualize>
-    <update_rate>5.0</update_rate>
-    <ray>
-      <scan>
-        <horizontal>
-        <samples>360</samples>
-        <resolution>1</resolution>
-        <min_angle>0.0</min_angle>
-        <max_angle>6.28319</max_angle>
-        </horizontal>
-      </scan>
-      <range>
-        <min>0.120</min>
-        <max>3.5</max>
-        <resolution>0.015</resolution>
-      </range>
-      <noise>
-        <type>gaussian</type>
-        <mean>0.0</mean>
-        <stddev>0.01</stddev>
-      </noise>
-    </ray>
-    <plugin name="gazebo_ros_lds_lfcd_controller" filename="libgazebo_ros_laser.so">
-      <topicName>/scan</topicName>
-      <frameName>base_scan</frameName>
-    </plugin>
-    </sensor>
-  </gazebo>
-  <carmodel/>
+  <willand/>
 </robot>
